Commit message: add meshes visual and collisions

File: servicebot_description/urdf/servicebot.urdf (robot description, URDF)
Before this commit: robot servicebot, 5 links, 4 joints
Links:
- removed link front_caster
- removed link front_wheel
- removed link left_wheel
- removed link right_wheel
- added link head_link, mass 1.0; collision sphere radius=0.13; visual mesh filename=package://servicebot_description/meshes/Head.obj
- added link head_pan_link, mass 1.0
- added link left_caster_wheel_link, mass 1.0; collision sphere radius=0.032; visual mesh filename=package://servicebot_description/meshes/CasterWheel_Left.obj
- added link left_foot_link, mass 1.0; collision box size=0.35 0.2 0.15; visual mesh filename=package://servicebot_description/meshes/CasterBracket_Left.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
- added link left_forearm_link, mass 1.0; collision cylinder length=0.3 radius=0.06; visual mesh filename=package://servicebot_description/meshes/Forearm_Left.obj
- added link left_upper_arm_link, mass 1.0; collision cylinder length=0.22 radius=0.065; visual mesh filename=package://servicebot_description/meshes/UpperArm_Left.obj
- added link left_upper_leg_link, mass 1.0; collision cylinder length=0.3 radius=0.12; visual mesh filename=package://servicebot_description/meshes/Calf_Left.obj
- added link left_wheel_link, mass 1.0; collision sphere radius=0.103; visual mesh filename=package://servicebot_description/meshes/Wheel_Left.obj
- added link pelvis_link, mass 1.0; collision cylinder length=0.20 radius=0.11; collision cylinder length=0.26 radius=0.12
- added link right_caster_wheel_link, mass 1.0; collision sphere radius=0.032; visual mesh filename=package://servicebot_description/meshes/CasterWheel_Left.obj
- added link right_foot_link, mass 1.0; collision box size=0.35 0.2 0.15; visual mesh filename=package://servicebot_description/meshes/CasterBracket_Left.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
- added link right_forearm_link, mass 1.0; collision cylinder length=0.3 radius=0.06; visual mesh filename=package://servicebot_description/meshes/Forearm_Right.obj
- added link right_upper_arm_link, mass 1.0; collision cylinder length=0.22 radius=0.065; visual mesh filename=package://servicebot_description/meshes/UpperArm_Left.obj
- added link right_upper_leg_link, mass 1.0; collision cylinder length=0.3 radius=0.12; visual mesh filename=package://servicebot_description/meshes/Calf_Right.obj
- added link right_wheel_link, mass 1.0; collision sphere radius=0.103; visual mesh filename=package://servicebot_description/meshes/Wheel_Left.obj
- link base_link: geometry collision box size=0.32 0.3 0.32; collision cylinder length=0.10 radius=0.07
Joints:
- removed joint front_caster_joint
- removed joint front_wheel_joint
- added joint head_pan_joint: type revolute, parent base_link, child head_pan_link, origin xyz=0 0.009 0.250 rpy=0 0 0, axis 0 0 -1, limit lower=-1.5707963267948966 upper=1.5707963267948966 effort=30 velocity=1.0
- added joint head_tilt_joint: type revolute, parent head_pan_link, child head_link, origin xyz=0 0 0 rpy=0 0 0, axis 0 -1 0, limit lower=-0.7853981633974483 upper=0.7853981633974483 effort=30 velocity=1.0
- added joint left_caster_wheel_joint: type continuous, parent left_foot_link, child left_caster_wheel_link, origin xyz=-0.14 0 -0.066 rpy=0 0 0, axis 0 1 0
- added joint left_elbow_fixedjoint: type fixed, parent left_upper_arm_link, child left_forearm_link, origin xyz=0.006 0.179 0 rpy=0 0 0
- added joint left_foot_fixedjoint: type fixed, parent left_upper_leg_link, child left_foot_link, origin xyz=0.041 0 -0.19 rpy=0 0 0
- added joint left_shoulder_fixedjoint: type fixed, parent base_link, child left_upper_arm_link, origin xyz=0 0.236 0.056 rpy=0 0 0
- added joint left_upper_leg_fixedjoint: type fixed, parent pelvis_link, child left_upper_leg_link, origin xyz=0.019 0.125 -0.256 rpy=0 0 0
- added joint pelvis_fixedjoint: type fixed, parent base_link, child pelvis_link, origin xyz=0 0.00 -0.286 rpy=0 0 0
- added joint right_caster_wheel_joint: type continuous, parent right_foot_link, child right_caster_wheel_link, origin xyz=-0.143 0 -0.064 rpy=0 0 0, axis 0 1 0
- added joint right_elbow_fixedjoint: type fixed, parent right_upper_arm_link, child right_forearm_link, origin xyz=0.006 -0.179 0 rpy=0 0 0
- added joint right_foot_fixedjoint: type fixed, parent right_upper_leg_link, child right_foot_link, origin xyz=0.041 0 -0.19 rpy=0 0 0
- added joint right_shoulder_fixedjoint: type fixed, parent base_link, child right_upper_arm_link, origin xyz=0 -0.236 0.056 rpy=0 0 0
- added joint right_upper_leg_fixedjoint: type fixed, parent pelvis_link, child right_upper_leg_link, origin xyz=0.019 -0.125 -0.256 rpy=0 0 0
- joint left_wheel_joint: axis 0 0 1 -> 0 1 0; child left_wheel -> left_wheel_link; origin xyz=-0.2825 0.125 -.15 rpy=-1.5708 0 0 -> xyz=0 0 0 rpy=0 0 0; parent base_link -> left_foot_link
- joint right_wheel_joint: axis 0 0 1 -> 0 1 0; child right_wheel -> right_wheel_link; origin xyz=-0.2825 -0.125 -.15 rpy=-1.5708 0 0 -> xyz=0 0 0 rpy=0 0 0; parent base_link -> right_foot_link

Commit message: add some gazebo tags for the links

File: servicebot_description/urdf/servicebot.urdf (robot description, URDF)
Before this commit: robot servicebot, 16 links, 15 joints
Joints:
- joint right_caster_wheel_joint: origin xyz=-0.143 0 -0.064 rpy=0 0 0 -> xyz=-0.14 0 -0.066 rpy=0 0 0

Commit message: Set mass and inertia for some links

File: servicebot_description/urdf/servicebot.urdf (robot description, URDF)
Before this commit: robot servicebot, 16 links, 15 joints
Links:
- link base_link: mass 1.0 -> 0.00001
- link head_link: mass 1.0 -> 0.5
- link head_pan_link: mass 1.0 -> 0.5
- link left_caster_wheel_link: mass 1.0 -> 0.03
- link left_foot_link: mass 1.0 -> 0.001
- link left_forearm_link: mass 1.0 -> 0.001
- link left_upper_arm_link: mass 1.0 -> 0.001
- link left_upper_leg_link: mass 1.0 -> 0.001
- link left_wheel_link: mass 1.0 -> 0.3
- link pelvis_link: mass 1.0 -> 0.001
- link right_caster_wheel_link: mass 1.0 -> 0.03
- link right_foot_link: mass 1.0 -> 0.001
- link right_forearm_link: mass 1.0 -> 0.001
- link right_upper_arm_link: mass 1.0 -> 0.001
- link right_upper_leg_link: mass 1.0 -> 0.001
- link right_wheel_link: mass 1.0 -> 0.3

Commit message: reexport all meshes manually and add joints

File: servicebot_description/urdf/servicebot.urdf (robot description, URDF)
Before this commit: robot servicebot, 16 links, 15 joints
Links:
- added link left_elbow_attach_link, mass 0.001; visual mesh filename=package://servicebot_description/meshes/Elbow_Left.obj
- added link left_hand_link, mass 0.001; collision box size=0.07 0.14 0.08; visual mesh filename=package://servicebot_description/meshes/Hand_Left.obj
- added link left_lower_hand_link, mass 0.001; collision box size=0.07 0.12 0.04; visual mesh filename=package://servicebot_description/meshes/LowerHand_Left.obj
- added link left_shoulder_link, mass 0.001; collision cylinder length=0.10 radius=0.08; visual mesh filename=package://servicebot_description/meshes/Shoulder_Left.obj
- added link left_thigh_link, mass 0.001; collision cylinder length=0.25 radius=0.12; visual mesh filename=package://servicebot_description/meshes/Thigh_Left.obj
- added link right_elbow_attach_link, mass 0.001; visual mesh filename=package://servicebot_description/meshes/Elbow_Left.obj
- added link right_hand_link, mass 0.001; collision box size=0.07 0.14 0.08; visual mesh filename=package://servicebot_description/meshes/Hand_Right.obj
- added link right_lower_hand_link, mass 0.001; collision box size=0.07 0.12 0.04; visual mesh filename=package://servicebot_description/meshes/LowerHand_Right.obj
- added link right_shoulder_link, mass 0.001; collision cylinder length=0.10 radius=0.08; visual mesh filename=package://servicebot_description/meshes/Shoulder_Right.obj
- added link right_thigh_link, mass 0.001; collision cylinder length=0.25 radius=0.12; visual mesh filename=package://servicebot_description/meshes/Thigh_Right.obj
- added link virtual_base_link; visual mesh filename=package://servicebot_description/meshes/servicebot.obj scale=0.01 0.01 0.01
- link base_link: geometry collision box size=0.32 0.3 0.32; collision cylinder length=0.10 radius=0.07
- link left_caster_wheel_link: geometry collision sphere radius=0.033; visual mesh filename=package://servicebot_description/meshes/CasterWheel_Left.obj
- link left_foot_link: geometry collision box size=0.35 0.2 0.15; visual mesh filename=package://servicebot_description/meshes/Foot_Left.obj
- link left_forearm_link: geometry collision cylinder length=0.16 radius=0.06; visual mesh filename=package://servicebot_description/meshes/Forearm_Left.obj
- link left_upper_arm_link: geometry collision cylinder length=0.15 radius=0.065; visual mesh filename=package://servicebot_description/meshes/UpperArm_Left.obj
- link left_upper_leg_link: geometry collision cylinder length=0.33 radius=0.12; visual mesh filename=package://servicebot_description/meshes/Calf_Left.obj
- link pelvis_link: geometry collision cylinder length=0.18 radius=0.1; visual mesh filename=package://servicebot_description/meshes/Pelvis.obj
- link right_caster_wheel_link: geometry collision sphere radius=0.033; visual mesh filename=package://servicebot_description/meshes/CasterWheel_Left.obj
- link right_forearm_link: geometry collision cylinder length=0.16 radius=0.06; visual mesh filename=package://servicebot_description/meshes/Forearm_Right.obj
- link right_upper_leg_link: geometry collision cylinder length=0.33 radius=0.12; visual mesh filename=package://servicebot_description/meshes/Calf_Left.obj
Joints:
- removed joint left_elbow_fixedjoint
- removed joint left_foot_fixedjoint
- removed joint left_shoulder_fixedjoint
- removed joint left_upper_leg_fixedjoint
- removed joint right_elbow_fixedjoint
- removed joint right_foot_fixedjoint
- removed joint right_shoulder_fixedjoint
- removed joint right_upper_leg_fixedjoint
- added joint left_elbow_attach_joint: type fixed, parent left_upper_arm_link, child left_elbow_attach_link, origin xyz=0 0.105 0.001 rpy=0 0 0
- added joint left_elbow_joint: type revolute, parent left_elbow_attach_link, child left_forearm_link, origin xyz=-0.006 0.055 -0.001 rpy=0 0 0, axis 0 0 1, limit lower=-0.5 upper=0 effort=30 velocity=1.0
- added joint left_foot_joint: type revolute, parent left_upper_leg_link, child left_foot_link, origin xyz=0.03 0 -0.335 rpy=0 0 0, axis 0 1 0, limit lower=-0.7853981633974483 upper=0.7853981633974483 effort=30 velocity=1.0
- added joint left_gripper_joint: type revolute, parent left_hand_link, child left_lower_hand_link, origin xyz=0.00 0.02 -0.025 rpy=0 0 0, axis 1 0 0, limit lower=-0.7853981633974483 upper=0 effort=30 velocity=1.0
- added joint left_hand_fixedjoint: type fixed, parent left_forearm_link, child left_hand_link, origin xyz=0.005 0.095 0.0 rpy=0 0 0
- added joint left_shoulder_joint: type revolute, parent base_link, child left_shoulder_link, origin xyz=0 0.1737 0.115 rpy=0 0 0, axis 0 1 0, limit lower=-0.7853981633974483 upper=0.7853981633974483 effort=30 velocity=1.0
- added joint left_thigh_joint: type revolute, parent pelvis_link, child left_thigh_link, origin xyz=0.017285 0.12 -0.11 rpy=0 0 0, axis 0 1 0, limit lower=-0.7853981633974483 upper=0.7853981633974483 effort=30 velocity=1.0
- added joint left_upper_arm_joint: type fixed, parent left_shoulder_link, child left_upper_arm_link, origin xyz=0 0.015 0.001 rpy=0 0 0
- added joint left_upper_leg_joint: type revolute, parent left_thigh_link, child left_upper_leg_link, origin xyz=0.011 0.005 -0.106 rpy=0 0 0, axis 0 1 0, limit lower=-0.15 upper=0.7853981633974483 effort=30 velocity=1.0
- added joint right_elbow_attach_joint: type fixed, parent right_upper_arm_link, child right_elbow_attach_link, origin xyz=0 -0.105 0.001 rpy=0 0 0
- added joint right_elbow_joint: type revolute, parent right_elbow_attach_link, child right_forearm_link, origin xyz=-0.006 -0.055 -0.001 rpy=0 0 0, axis 0 0 -1, limit lower=-0.5 upper=0 effort=30 velocity=1.0
- added joint right_foot_joint: type revolute, parent right_upper_leg_link, child right_foot_link, origin xyz=0.03 0 -0.335 rpy=0 0 0, axis 0 1 0, limit lower=-0.7853981633974483 upper=0.7853981633974483 effort=30 velocity=1.0
- added joint right_gripper_joint: type revolute, parent right_hand_link, child right_lower_hand_link, origin xyz=0.00 -0.02 -0.025 rpy=0 0 0, axis -1 0 0, limit lower=-0.7853981633974483 upper=0 effort=30 velocity=1.0
- added joint right_hand_fixedjoint: type fixed, parent right_forearm_link, child right_hand_link, origin xyz=0.005 -0.095 0.0 rpy=0 0 0
- added joint right_shoulder_joint: type revolute, parent base_link, child right_shoulder_link, origin xyz=0 -0.1737 0.115 rpy=0 0 0, axis 0 1 0, limit lower=-0.7853981633974483 upper=0.7853981633974483 effort=30 velocity=1.0
- added joint right_thigh_joint: type revolute, parent pelvis_link, child right_thigh_link, origin xyz=0.017285 -0.12 -0.11 rpy=0 0 0, axis 0 1 0, limit lower=-0.7853981633974483 upper=0.7853981633974483 effort=30 velocity=1.0
- added joint right_upper_arm_joint: type fixed, parent right_shoulder_link, child right_upper_arm_link, origin xyz=0 -0.015 0.001 rpy=0 0 0
- added joint right_upper_leg_joint: type revolute, parent right_thigh_link, child right_upper_leg_link, origin xyz=0.011 -0.005 -0.106 rpy=0 0 0, axis 0 1 0, limit lower=-0.15 upper=0.7853981633974483 effort=30 velocity=1.0
- added joint virtual_base_fixedjoint: type fixed, parent virtual_base_link, child base_link, origin xyz=0 0.0 0.772 rpy=0 0 0
- joint head_pan_joint: origin xyz=0 0.009 0.250 rpy=0 0 0 -> xyz=0 0 0.31 rpy=0 0 0
- joint left_caster_wheel_joint: origin xyz=-0.14 0 -0.066 rpy=0 0 0 -> xyz=-0.142 0 -0.07 rpy=0 0 0
- joint pelvis_fixedjoint: origin xyz=0 0.00 -0.286 rpy=0 0 0 -> xyz=0 0.00 -0.12 rpy=0 0 0

Commit message: make leg joint fixed in the current default pose

File: servicebot_description/urdf/servicebot.urdf (robot description, URDF)
Before this commit: robot servicebot, 27 links, 26 joints
Links:
- removed link virtual_base_link
- link base_link: mass 0.00001 -> 3
- link left_elbow_attach_link: mass 0.001 -> 0.15
- link left_forearm_link: mass 0.001 -> 0.2
- link left_hand_link: mass 0.001 -> 0.1
- link left_lower_hand_link: mass 0.001 -> 0.1
- link left_thigh_link: mass 0.001 -> 1
- link left_upper_arm_link: mass 0.001 -> 0.2
- link left_upper_leg_link: mass 0.001 -> 0.5
- link pelvis_link: mass 0.001 -> 1
- link right_elbow_attach_link: mass 0.001 -> 0.15
- link right_foot_link: geometry collision box size=0.35 0.2 0.15; visual mesh filename=package://servicebot_description/meshes/Foot_Left.obj
- link right_forearm_link: mass 0.001 -> 0.2
- link right_hand_link: mass 0.001 -> 0.1
- link right_lower_hand_link: mass 0.001 -> 0.1
- link right_thigh_link: mass 0.001 -> 1
- link right_upper_arm_link: mass 0.001 -> 0.2
- link right_upper_leg_link: mass 0.001 -> 0.5
Joints:
- removed joint virtual_base_fixedjoint
- joint left_elbow_joint: limit lower=-0.5 upper=0 effort=30 velocity=1.0 -> lower=-0.5 upper=-0.5 effort=30 velocity=1.0
- joint left_foot_joint: axis 0 1 0 -> (none); limit lower=-0.7853981633974483 upper=0.7853981633974483 effort=30 velocity=1.0 -> (none); origin xyz=0.03 0 -0.335 rpy=0 0 0 -> xyz=0.03 0 -0.335 rpy=0.000 -0.160 0.000; type revolute -> fixed
- joint left_shoulder_joint: limit lower=-0.7853981633974483 upper=0.7853981633974483 effort=30 velocity=1.0 -> lower=-0.55 upper=-00.55 effort=30 velocity=1.0
- joint left_thigh_joint: axis 0 1 0 -> (none); limit lower=-0.7853981633974483 upper=0.7853981633974483 effort=30 velocity=1.0 -> (none); origin xyz=0.017285 0.12 -0.11 rpy=0 0 0 -> xyz=0.017285 0.12 -0.11 rpy=0.000 -0.640 0.000; type revolute -> fixed
- joint left_upper_arm_joint: axis (none) -> -1 0 0; limit (none) -> lower=1.35 upper=1.35 effort=30 velocity=1.0; type fixed -> revolute
- joint left_upper_leg_joint: limit lower=-0.15 upper=0.7853981633974483 effort=30 velocity=1.0 -> (none); origin xyz=0.011 0.005 -0.106 rpy=0 0 0 -> xyz=0.011 0.005 -0.106 rpy=0.000 0.785 0.000; type revolute -> fixed
- joint right_caster_wheel_joint: origin xyz=-0.14 0 -0.066 rpy=0 0 0 -> xyz=-0.142 0 -0.07 rpy=0 0 0
- joint right_elbow_joint: limit lower=-0.5 upper=0 effort=30 velocity=1.0 -> lower=-0.5 upper=-0.5 effort=30 velocity=1.0
- joint right_foot_joint: axis 0 1 0 -> (none); limit lower=-0.7853981633974483 upper=0.7853981633974483 effort=30 velocity=1.0 -> (none); origin xyz=0.03 0 -0.335 rpy=0 0 0 -> xyz=0.03 0 -0.335 rpy=0.000 -0.160 0.000; type revolute -> fixed
- joint right_shoulder_joint: limit lower=-0.7853981633974483 upper=0.7853981633974483 effort=30 velocity=1.0 -> lower=-0.55 upper=-0.55 effort=30 velocity=1.0
- joint right_thigh_joint: axis 0 1 0 -> (none); limit lower=-0.7853981633974483 upper=0.7853981633974483 effort=30 velocity=1.0 -> (none); origin xyz=0.017285 -0.12 -0.11 rpy=0 0 0 -> xyz=0.017285 -0.12 -0.11 rpy=0.000 -0.640 0.000; type revolute -> fixed
- joint right_upper_arm_joint: axis (none) -> 1 0 0; limit (none) -> lower=1.35 upper=1.35 effort=30 velocity=1.0; type fixed -> revolute
- joint right_upper_leg_joint: limit lower=-0.15 upper=0.7853981633974483 effort=30 velocity=1.0 -> (none); origin xyz=0.011 -0.005 -0.106 rpy=0 0 0 -> xyz=0.011 -0.005 -0.106 rpy=0.000 0.785 0.000; type revolute -> fixed

Commit message: WIP add max acceleration to wheels, a front camera frame, a camera sensor and controllers for the head joints

File: servicebot_description/urdf/servicebot.urdf (robot description, URDF)
Before this commit: robot servicebot, 26 links, 25 joints
Links:
- added link front_camera_frame, mass 0.001
Joints:
- added joint front_camera_fixedjoint: type fixed, parent head_link, child front_camera_frame, origin xyz=0.1 0 0 rpy=0 0 0
- joint head_pan_joint: limit lower=-1.5707963267948966 upper=1.5707963267948966 effort=30 velocity=1.0 -> lower=-1.5707963267948966 upper=1.5707963267948966 effort=200 velocity=1.0
- joint head_tilt_joint: limit lower=-0.7853981633974483 upper=0.7853981633974483 effort=30 velocity=1.0 -> lower=-0.7853981633974483 upper=0.7853981633974483 effort=200 velocity=1.0

Commit message: update configuration files, fix arm links, publish caster wheel joints, add sensors

File: servicebot_description/urdf/servicebot.urdf (robot description, URDF)
Before this commit: robot servicebot, 27 links, 26 joints
Links:
- added link front_camera_optical_frame, mass 0.001
- added link lidar_frame, mass 0.001
- added link rear_camera_frame, mass 0.001
- added link rear_camera_optical_frame, mass 0.001
Joints:
- removed joint right_thigh_joint
- added joint front_camera_optical_fixedjoint: type fixed, parent front_camera_frame, child front_camera_optical_frame, origin xyz=0 0 0 rpy=-1.57079632679 0 -1.57079632679
- added joint neck_lidar_fixedjoint: type fixed, parent base_link, child lidar_frame, origin xyz=0.05 0 0.22 rpy=0 0 0
- added joint rear_camera_fixedjoint: type fixed, parent head_link, child rear_camera_frame, origin xyz=-0.1 0 0 rpy=0 0 3.14159265
- added joint rear_camera_optical_fixedjoint: type fixed, parent rear_camera_frame, child rear_camera_optical_frame, origin xyz=0 0 0 rpy=-1.57079632679 0 -1.57079632679
- added joint right_thigh_joint/: type fixed, parent pelvis_link, child right_thigh_link, origin xyz=0.017285 -0.12 -0.11 rpy=0.000 -0.640 0.000
- joint head_pan_joint: origin xyz=0 0 0.31 rpy=0 0 0 -> xyz=0 0 0.32 rpy=0 0 0
- joint left_elbow_joint: axis 0 0 1 -> (none); limit lower=-0.5 upper=-0.5 effort=30 velocity=1.0 -> (none); origin xyz=-0.006 0.055 -0.001 rpy=0 0 0 -> xyz=-0.006 0.055 -0.001 rpy=0 0 -0.50; type revolute -> fixed
- joint left_gripper_joint: axis 1 0 0 -> (none); limit lower=-0.7853981633974483 upper=0 effort=30 velocity=1.0 -> (none); type revolute -> fixed
- joint left_shoulder_joint: axis 0 1 0 -> (none); limit lower=-0.55 upper=-00.55 effort=30 velocity=1.0 -> (none); origin xyz=0 0.1737 0.115 rpy=0 0 0 -> xyz=0 0.1737 0.115 rpy=0 -0.55 0; type revolute -> fixed
- joint left_upper_arm_joint: axis -1 0 0 -> (none); limit lower=1.35 upper=1.35 effort=30 velocity=1.0 -> (none); origin xyz=0 0.015 0.001 rpy=0 0 0 -> xyz=0 0.015 0.001 rpy=-1.35 0 0; type revolute -> fixed
- joint right_elbow_joint: axis 0 0 -1 -> (none); limit lower=-0.5 upper=-0.5 effort=30 velocity=1.0 -> (none); origin xyz=-0.006 -0.055 -0.001 rpy=0 0 0 -> xyz=-0.006 -0.055 -0.001 rpy=0 0 0.5; type revolute -> fixed
- joint right_gripper_joint: axis -1 0 0 -> (none); limit lower=-0.7853981633974483 upper=0 effort=30 velocity=1.0 -> (none); type revolute -> fixed
- joint right_shoulder_joint: axis 0 1 0 -> (none); limit lower=-0.55 upper=-0.55 effort=30 velocity=1.0 -> (none); origin xyz=0 -0.1737 0.115 rpy=0 0 0 -> xyz=0 -0.1737 0.115 rpy=0 -0.55 0; type revolute -> fixed
- joint right_upper_arm_joint: axis 1 0 0 -> (none); limit lower=1.35 upper=1.35 effort=30 velocity=1.0 -> (none); origin xyz=0 -0.015 0.001 rpy=0 0 0 -> xyz=0 -0.015 0.001 rpy=1.35 0 0; type revolute -> fixed

Commit message: tune physics params and use effort controllers

File: servicebot_description/urdf/servicebot.urdf (robot description, URDF)
Before this commit: robot servicebot, 31 links, 30 joints
Joints:
- joint head_pan_joint: limit lower=-1.5707963267948966 upper=1.5707963267948966 effort=200 velocity=1.0 -> lower=-1.5707963267948966 upper=1.5707963267948966 effort=30 velocity=1.0
- joint head_tilt_joint: limit lower=-0.7853981633974483 upper=0.7853981633974483 effort=200 velocity=1.0 -> lower=-0.7853981633974483 upper=0.7853981633974483 effort=30 velocity=1.0

Commit message: more fixups

File: servicebot_description/urdf/servicebot.urdf (robot description, URDF)
Before this commit: robot servicebot, 31 links, 30 joints
Joints:
- removed joint right_thigh_joint/
- added joint right_thigh_joint: type fixed, parent pelvis_link, child right_thigh_link, origin xyz=0.017285 -0.12 -0.11 rpy=0.000 -0.640 0.000

Commit message: Approximation penalty

File: servicebot_description/urdf/servicebot.urdf (robot description, URDF)
Before this commit: robot servicebot, 31 links, 30 joints
Links:
- link base_link: geometry collision box size=0.32 0.3 0.32; collision cylinder length=0.10 radius=0.07

Commit message: collide_without_contact on URDF, reduce spam, fit through doors

File: servicebot_description/urdf/servicebot.urdf (robot description, URDF)
Before this commit: robot servicebot, 31 links, 30 joints
Links:
- added link inflation_obj, mass 0.001; collision cylinder length=1.07 radius=0.35
- added link inflation_people, mass 0.001; collision cylinder length=1.07 radius=0.75
- link base_link: geometry collision box size=0.32 0.3 0.32; collision cylinder length=0.10 radius=0.07
Joints:
- added joint inflation_obj_fixedjoint: type fixed, parent base_link, child inflation_obj
- added joint inflation_people_fixedjoint: type fixed, parent base_link, child inflation_people
