Commit message: added base_footprint, tighter amcl config, and better rviz config

File: servicebot_description/urdf/servicebot.urdf (robot description, URDF)
Before this commit: robot servicebot, 33 links, 32 joints
Links:
- added link base_footprint
Joints:
- added joint base_footprint_joint: type fixed, parent base_footprint, child base_link, origin xyz=0 0 0.749 rpy=0 0 0
